Commit message: adding ur baseline to core.launch.py for plugin:=mock and gripper:=none,crab_claw

File: ur_simulation_gz/urdf/ur_bam_eef.urdf.xacro (robot description, xacro)
@@ -73,19 +73,26 @@
   </gazebo>
   <!-- ros2 control instance -->
+  <!-- Adding plugin to allow for mock -->
+  <xacro:arg name="plugin" default="mock"/>  <!-- none, mock, gazebo, real -->
   <xacro:ur_ros2_control
     name="$(arg name)"
     tf_prefix="$(arg tf_prefix)"
+    plugin="$(arg plugin)"
     transmission_hw_interface="$(arg transmission_hw_interface)"
   />
   <!-- ABOVE IS COPIED PASTED FROM ur_gz.urdf.xacro, add bam_gripper below-->
-    <joint name="$(arg tf_prefix)tool0-eef_link_1" type="fixed">
+  <xacro:arg name="gripper" default="" />
+  <xacro:property name="gripper" value="$(arg gripper)"/>
+  <xacro:include filename="$(find bam_descriptions)/urdf/common.xacro" />
+  <xacro:if value="${gripper == 'crab_claw'}">
+      <joint name="$(arg tf_prefix)tool0-eef_link_1" type="fixed">
       <parent link="$(arg tf_prefix)tool0" />
       <child link="eef_link_1" />
       <origin xyz="0 0 0" rpy="0 0 0" />
     </joint>
-  <xacro:include filename="$(find bam_descriptions)/urdf/common.xacro" />
-  <xacro:include filename="$(find bam_descriptions)/urdf/gripper_v1/gripper_v1_macro.xacro" />
-  <xacro:gripper_v1 prefix="" reflect="1"/>
-  <xacro:include filename="$(find bam_descriptions)/urdf/gripper_v1/gripper_v1.ros2_control.xacro" />
-  <xacro:gripper_v1_ros2_control prefix="" plugin="gazebo"/>
+    <xacro:include filename="$(find bam_descriptions)/urdf/gripper_v1/gripper_v1_macro.xacro" />
+    <xacro:gripper_v1 prefix="" reflect="1"/>
+    <xacro:include filename="$(find bam_descriptions)/urdf/gripper_v1/gripper_v1.ros2_control.xacro" />
+    <xacro:gripper_v1_ros2_control prefix="" plugin="gazebo"/>
+  </xacro:if>
 </robot>

File: ur_simulation_gz/urdf/ur_gz.ros2_control.xacro (robot description, xacro)
@@ -5,4 +5,5 @@
     name
     tf_prefix
+    plugin
     transmission_hw_interface:=hardware_interface/PositionJointInterface
     initial_positions:=${dict(shoulder_pan_joint=0.0,shoulder_lift_joint=-1.57,elbow_joint=0.0,wrist_1_joint=-1.57,wrist_2_joint=0.0,wrist_3_joint=0.0)}
@@ -13,5 +14,10 @@
     <ros2_control name="${name}" type="system">
       <hardware>
-        <plugin>gz_ros2_control/GazeboSimSystem</plugin>
+        <xacro:if value="${plugin == 'gazebo'}">
+            <plugin>gz_ros2_control/GazeboSimSystem</plugin>
+        </xacro:if>
+        <xacro:unless value="${plugin == 'gazebo'}">
+            <plugin>mock_components/GenericSystem</plugin>
+        </xacro:unless>
       </hardware>
       <xacro:ur_joint_control_description

Commit message: gripper working better now!

File: ur_simulation_gz/urdf/ur_bam_eef.urdf.xacro (robot description, xacro)
@@ -86,5 +86,5 @@
   <xacro:include filename="$(find bam_descriptions)/urdf/common.xacro" />
   <xacro:if value="${gripper == 'crab_claw'}">
-      <joint name="$(arg tf_prefix)tool0-eef_link_1" type="fixed">
+      <joint name="$(arg tf_prefix)tool0_to_eef_link_1" type="fixed">
       <parent link="$(arg tf_prefix)tool0" />
       <child link="eef_link_1" />

Commit message: ss

File: ur_simulation_gz/urdf/ur_bam_eef.urdf.xacro (robot description, xacro)
@@ -18,5 +18,6 @@
   <xacro:arg name="transmission_hw_interface" default=""/>
   <xacro:arg name="safety_limits" default="false"/>
-  <xacro:arg name="safety_pos_margin" default="0.15"/>
+  <!-- <xacro:arg name="safety_pos_margin" default="0.15"/> -->
+  <xacro:arg name="safety_pos_margin" default="0.0"/>
   <xacro:arg name="safety_k_position" default="20"/>
   <xacro:arg name="simulation_controllers" default="" />
@@ -24,5 +25,5 @@
   <!-- create link fixed to the "world" -->
   <link name="world" />
-  <link name="ground_plane">
+  <!-- <link name="ground_plane">
     <visual>
       <origin rpy="0 0 0" xyz="0 0 0"/>
@@ -45,5 +46,5 @@
     <parent link="world"/>
     <child link="ground_plane"/>
-  </joint>
+  </joint> -->
   <!-- arm -->
   <xacro:ur_robot

File: ur_simulation_gz/urdf/ur_gz.urdf.xacro (robot description, xacro)
@@ -17,5 +17,6 @@
   <xacro:arg name="transmission_hw_interface" default=""/>
   <xacro:arg name="safety_limits" default="false"/>
-  <xacro:arg name="safety_pos_margin" default="0.15"/>
+  <xacro:arg name="safety_pos_margin" default="0.0"/>
+  <!-- <xacro:arg name="safety_pos_margin" default="0.15"/> -->
   <xacro:arg name="safety_k_position" default="20"/>
   <xacro:arg name="simulation_controllers" default="" />
@@ -23,5 +24,5 @@
   <!-- create link fixed to the "world" -->
   <link name="world" />
-  <link name="ground_plane">
+  <!-- <link name="ground_plane">
     <visual>
       <origin rpy="0 0 0" xyz="0 0 0"/>
@@ -44,5 +45,5 @@
     <parent link="world"/>
     <child link="ground_plane"/>
-  </joint>
+  </joint> -->
   <!-- arm -->
   <xacro:ur_robot
